File: Platine/Tonuino V1.0.sch (EAGLE design)
At the start: 32 parts, among them T1 BC857, T2 BC847, T3 BC847, T4 IRLML2502

Commit message: Add files via upload
Parts:
- removed OP_ON, PWR, WAKE: (no value), pinhead:PINHD-1X2
- removed STATUS: (no value), led:LED5MM
- added AKKU, JP1, JP2, OP_H, OP_L, PB, WK1, WK2: (no value), pinhead:PINHD-1X2
- added C2: 33n, rcl:C-EUC0805
- added P_SEL: (no value), pinhead:PINHD-1X3
- added R10: 100, rcl:R-EU_R1206
- added R11: 3M, rcl:R-EU_R1206
- added R12: 2,5k, rcl:R-EU_R1206
- added STAT: (no value), led:LED5MM
- added T5: IRLML2502, transistor-fet:IRLML2502
- added T6: BC847, transistor:BC847
- C1: value (none) -> 220µF
Connections:
- new net N$16: R8.2, STAT.C
- new net N$17: ARDUINO_NANO.D8, JP2.1
- new net N$20: PB.2, R11.2, T5.D
- new net PWR_ON_PIN_JPR: ARDUINO_NANO.D7, JP1.1
- new net VCC_AKKU: P_SEL.3, T4.S
- new net VCC_PB: P_SEL.1, T5.S
- net GND: now also AKKU.1, C2.2, OP_H.1, OP_L.1, PB.1, R10.1, R8.1, T6.E, WK2.1; no longer OP_ON.1, PWR.1, STATUS.C
- net N$10: now also JP2.2, OP_H.2, T6.C; no longer OP_ON.2
- net N$22: now also STAT.A; no longer R8.2
- net N$23: now also OP_L.2, R12.2, T6.B; no longer R8.1, STATUS.A
- net N$25: now also R10.2, WK1.1; no longer WAKE.1
- net PWR_ON_PIN: now also JP1.2; no longer ARDUINO_NANO.D7
- net TASTER: now also C2.1, R11.1, T5.G, WK2.2
- net VCC: now also AKKU.2, WK1.2; no longer PWR.2, WAKE.2
- net VCC_TONUINO: now also P_SEL.2, R12.1; no longer T4.S
Other:
- note added: "AKKU: Stromversorgung über Akku"
- note added: "Akku Power Management"
- note added: "JP1: --D7-- PWR_ON_PIN (Selbsthaltung durch µC)"
- note added: "JP2: --D8-- OP_ON (Kopfhörerbuchsen-Überwachung durch µC)"
- note added: "OP_H: Steuerung Lautsprecherverstärker (gebrückt: OP EIN)"
- note added: "OP_L: Steuerung Lautsprecherverstärker (gebrückt: OP AUS)"
- note added: "PB: Stromversorgung über PowerBank"
- note added: "P_SEL: Auswahl der Stromversorgung (entw. Powerbank oder Akku)"
- note added: "PowerSource Selection"
- note added: "WK1: WakeUp-Kontakt für Akku-Betrieb"
- note added: "WK2: WakeUp-Kontakt für Betrieb über Powerbank"
- moved on the sheet: 3,3V, 5V, ARDUINO_NANO, C1, D1, D2, D3, D4, EAR, GND, R1, R2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
